File: test123.kicad_sch (KiCad schematic)
At the start: 15 parts, among them J2 XH-8A, J3 Conn_01x06, J4 Conn_01x35, J5 Conn_01x35, J6 Conn_01x23, M1 Module-wbo-0.2, M2 Module-can-0.1, P1 Pad, Q1 ISL9V3040S3S

Commit message: Signed-off-by: J62 <j.owens@interbiznw.com>
Parts:
- gave numbers to parts that had none: 1
